Commit message: 6.6 Gazrbo

File: src/urdf02_gazebo/xacro/my_base.urdf.xacro (robot description, xacro)
@@ -9,5 +9,6 @@
 <robot name="my_base" xmlns:xacro="http://www.ros.org/wiki/xacro">
     <!-- 封装变量、常量 -->
-    <xacro:property name="PI" value="3.141"/>
+    <!-- PI 值设置精度需要高一些，否则后续车轮翻转量计算时，可能会出现肉眼不能察觉的车轮倾斜，从而导致模型抖动 -->
+    <xacro:property name="PI" value="3.1415926"/>
     <!-- 宏:黑色设置 -->
     <material name="black">
@@ -19,4 +20,5 @@
     <xacro:property name="base_link_length" value="0.08" /> <!-- base_link 长 -->
     <xacro:property name="earth_space" value="0.015" /> <!-- 离地间距 -->
+    <xacro:property name="base_link_m" value="0.5" /> <!-- 质量  -->
     <!-- 底盘 -->
     <link name="base_footprint">
@@ -37,4 +39,11 @@
         </material>
       </visual>
+      <collision>
+        <geometry>
+          <cylinder radius="${base_link_radius}" length="${base_link_length}" />
+        </geometry>
+        <origin xyz="0 0 0" rpy="0 0 0" />
+      </collision>
+      <xacro:cylinder_inertial_matrix m="${base_link_m}" r="${base_link_radius}" h="${base_link_length}" />
     </link>
     <joint name="base_link2base_footprint" type="fixed">
@@ -43,10 +52,14 @@
       <origin xyz="0 0 ${earth_space + base_link_length / 2 }" />
     </joint>
+    <gazebo reference="base_link">
+        <material>Gazebo/Yellow</material>
+    </gazebo>
     <!-- 驱动轮 -->
     <!-- 驱动轮属性 -->
     <xacro:property name="wheel_radius" value="0.0325" /><!-- 半径 -->
     <xacro:property name="wheel_length" value="0.015" /><!-- 宽度 -->
+    <xacro:property name="wheel_m" value="0.05" /> <!-- 质量  -->
     <!-- 驱动轮宏实现 -->
-    <xacro:macro name="add_wheels" params="name flag joint_name">
+    <xacro:macro name="add_wheels" params="name flag">
       <link name="${name}_wheel">
         <visual>
@@ -57,17 +70,28 @@
           <material name="black" />
         </visual>
+        <collision>
+          <geometry>
+            <cylinder radius="${wheel_radius}" length="${wheel_length}" />
+          </geometry>
+          <origin xyz="0.0 0.0 0.0" rpy="${PI / 2} 0.0 0.0" />
+        </collision>
+        <xacro:cylinder_inertial_matrix m="${wheel_m}" r="${wheel_radius}" h="${wheel_length}" />
       </link>
-      <joint name="${joint_name}" type="continuous">
+      <joint name="${name}_wheel2base_link" type="continuous">
         <parent link="base_link" />
         <child link="${name}_wheel" />
-        <origin xyz="0 ${flag * (base_link_radius + wheel_length / 2)} ${-(earth_space + base_link_length / 2 - wheel_radius) }" />
+        <origin xyz="0 ${flag * base_link_radius} ${-(earth_space + base_link_length / 2 - wheel_radius) }" />
         <axis xyz="0 1 0" />
       </joint>
+      <gazebo reference="${name}_wheel">
+        <material>Gazebo/Red</material>
+      </gazebo>
     </xacro:macro>
-    <xacro:add_wheels name="left" flag="1" joint_name="base_l_wheel_joint" />
-    <xacro:add_wheels name="right" flag="-1" joint_name="base_r_wheel_joint" />
+    <xacro:add_wheels name="left" flag="1" />
+    <xacro:add_wheels name="right" flag="-1" />
     <!-- 支撑轮 -->
     <!-- 支撑轮属性 -->
     <xacro:property name="support_wheel_radius" value="0.0075" /> <!-- 支撑轮半径 -->
+    <xacro:property name="support_wheel_m" value="0.03" /> <!-- 质量  -->
     <!-- 支撑轮宏 -->
     <xacro:macro name="add_support_wheel" params="name flag" >
@@ -80,4 +104,11 @@
             <material name="black" />
         </visual>
+        <collision>
+            <geometry>
+                <sphere radius="${support_wheel_radius}" />
+            </geometry>
+            <origin xyz="0 0 0" rpy="0 0 0" />
+        </collision>
+        <xacro:sphere_inertial_matrix m="${support_wheel_m}" r="${support_wheel_radius}" />
       </link>
       <joint name="${name}_wheel2base_link" type="continuous">
@@ -87,4 +118,7 @@
           <axis xyz="1 1 1" />
       </joint>
+      <gazebo reference="${name}_wheel">
+        <material>Gazebo/Red</material>
+      </gazebo>
     </xacro:macro>
     <xacro:add_support_wheel name="front" flag="1" />
